File: Electrical/NMEA-2000-BUS-Voltage.kicad_sch (KiCad schematic)
At the start: 0 parts

Commit message: Added D1 Mini to Schematic
Parts:
- added U1: WeMos_D1_mini, Module:WEMOS_D1_mini_light, symbol MCU_Module:WeMos_D1_mini
Connections:
- new net +3V3: U1.8 (3V3)
- new net +5V: U1.9 (5V)
- new net A0: U1.2 (A0)
- new net D1: U1.14 (SCL/D1)
- new net FLS: U1.12 (D3)
- new net GND: U1.10 (GND)
- new net RX: U1.15 (RX)
- new net TX: U1.16 (TX)
- no-connect marks 0 -> 8
Changed lines of the file:
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@@
 (kicad_sch (version 20230121) (generator eeschema)
   (paper "A4")
+  (no_connect (at 64.77 102.87))
+  (no_connect (at 64.77 87.63))
+  (no_connect (at 64.77 92.71))
+  (no_connect (at 64.77 100.33))
+  (no_connect (at 34.29 87.63))
+  (no_connect (at 64.77 97.79))
+  (no_connect (at 64.77 107.95))
+  (no_connect (at 64.77 105.41))
+  (wire (pts (xy 34.29 87.63) (xy 39.37 87.63))
+    (stroke (width 0) (type default))
+  )
+  (wire (pts (xy 46.99 74.93) (xy 46.99 77.47))
+    (stroke (width 0) (type default))
+  )
+  (wire (pts (xy 59.69 90.17) (xy 64.77 90.17))
+    (stroke (width 0) (type default))
+  )
+  (wire (pts (xy 64.77 105.41) (xy 59.69 105.41))
+    (stroke (width 0) (type default))
+  )
+  (wire (pts (xy 64.77 97.79) (xy 59.69 97.79))
+    (stroke (width 0) (type default))
+  )
+  (wire (pts (xy 64.77 87.63) (xy 59.69 87.63))
+    (stroke (width 0) (type default))
+  )
+  (wire (pts (xy 64.77 100.33) (xy 59.69 100.33))
+    (stroke (width 0) (type default))
+  )
+  (wire (pts (xy 34.29 97.79) (xy 39.37 97.79))
+    (stroke (width 0) (type default))
+  )
+  (wire (pts (xy 64.77 92.71) (xy 59.69 92.71))
+    (stroke (width 0) (type default))
+  )
+  (wire (pts (xy 52.07 74.93) (xy 52.07 77.47))
+    (stroke (width 0) (type default))
+  )
+  (wire (pts (xy 49.53 118.11) (xy 49.53 120.65))
+    (stroke (width 0) (type default))
+  )
+  (wire (pts (xy 59.69 95.25) (xy 64.77 95.25))
+    (stroke (width 0) (type default))
+  )
+  (wire (pts (xy 59.69 85.09) (xy 64.77 85.09))
+    (stroke (width 0) (type default))
+  )
+  (wire (pts (xy 64.77 102.87) (xy 59.69 102.87))
+    (stroke (width 0) (type default))
+  )
+  (wire (pts (xy 34.29 95.25) (xy 39.37 95.25))
+    (stroke (width 0) (type default))
+  )
+  (wire (pts (xy 64.77 107.95) (xy 59.69 107.95))
+    (stroke (width 0) (type default))
+  )
+  (label "TX" (at 34.29 97.79 0) (fields_autoplaced)
+    (effects (font (size 1.27 1.27)) (justify left bottom))
+  )
+  (label "A0" (at 64.77 85.09 180) (fields_autoplaced)
+    (effects (font (size 1.27 1.27)) (justify right bottom))
+  )
+  (label "FLS" (at 64.77 95.25 180) (fields_autoplaced)
+    (effects (font (size 1.27 1.27)) (justify right bottom))
+  )
+  (label "RX" (at 34.29 95.25 0) (fields_autoplaced)
+    (effects (font (size 1.27 1.27)) (justify left bottom))
+  )
+  (label "D1" (at 64.77 90.17 180) (fields_autoplaced)
+    (effects (font (size 1.27 1.27)) (justify right bottom))
+  )
+  (symbol (lib_id "MCU_Module:WeMos_D1_mini") (at 49.53 97.79 0) (unit 1)
+    (in_bom yes) (on_board yes) (dnp no) (fields_autoplaced)
+    (property "Reference" "U1" (at 51.4859 118.11 0)
+      (effects (font (size 1.27 1.27)) (justify left))
+    )
+    (property "Value" "WeMos_D1_mini" (at 51.4859 120.65 0)
+      (effects (font (size 1.27 1.27)) (justify left))
+    )
+    (property "Footprint" "Module:WEMOS_D1_mini_light" (at 49.53 127 0)
+      (effects (font (size 1.27 1.27)) hide)
+    )
+    (property "Datasheet" "https://wiki.wemos.cc/products:d1:d1_mini#documentation" (at 2.54 127 0)
+      (effects (font (size 1.27 1.27)) hide)
+    )
+    (pin "1")
+    (pin "10")
+    (pin "11")
+    (pin "12")
+    (pin "13")
+    (pin "14")
+    (pin "15")
+    (pin "16")
+    (pin "2")
+    (pin "3")
+    (pin "4")
+    (pin "5")
+    (pin "6")
+    (pin "7")
+    (pin "8")
+    (pin "9")
+    (instances
+      (project "NMEA-2000-BUS-Voltage"
+        (path "/2ad9a196-bb2f-4407-b356-e110a1476183"
+          (reference "U1") (unit 1)
+        )
+      )
+    )
+  )
+  (symbol (lib_id "power:+3V3") (at 52.07 74.93 0) (unit 1)
+    (in_bom yes) (on_board yes) (dnp no) (fields_autoplaced)
+    (property "Reference" "#PWR02" (at 52.07 78.74 0)
+      (effects (font (size 1.27 1.27)) hide)
+    )
+    (property "Value" "+3V3" (at 52.07 69.85 0)
+      (effects (font (size 1.27 1.27)))
+    )
+    (property "Footprint" "" (at 52.07 74.93 0)
+      (effects (font (size 1.27 1.27)) hide)
+    )
+    (property "Datasheet" "" (at 52.07 74.93 0)
+      (effects (font (size 1.27 1.27)) hide)
+    )
+    (pin "1")
+    (instances
+      (project "NMEA-2000-BUS-Voltage"
+        (path "/2ad9a196-bb2f-4407-b356-e110a1476183"
+          (reference "#PWR02") (unit 1)
+        )
+      )
+    )
+  )
+  (symbol (lib_id "power:GND") (at 49.53 120.65 0) (unit 1)
+    (in_bom yes) (on_board yes) (dnp no) (fields_autoplaced)
+    (property "Reference" "#PWR01" (at 49.53 127 0)
+      (effects (font (size 1.27 1.27)) hide)
+    )
+    (property "Value" "GND" (at 49.53 125.73 0)
+      (effects (font (size 1.27 1.27)))
+    )
+    (property "Footprint" "" (at 49.53 120.65 0)
+      (effects (font (size 1.27 1.27)) hide)
+    )
+    (property "Datasheet" "" (at 49.53 120.65 0)
+      (effects (font (size 1.27 1.27)) hide)
+    )
+    (pin "1")
+    (instances
+      (project "NMEA-2000-BUS-Voltage"
+        (path "/2ad9a196-bb2f-4407-b356-e110a1476183"
+          (reference "#PWR01") (unit 1)
+        )
+      )
+    )
+  )
+  (symbol (lib_id "power:+5V") (at 46.99 74.93 0) (unit 1)
+    (in_bom yes) (on_board yes) (dnp no) (fields_autoplaced)
+    (property "Reference" "#PWR03" (at 46.99 78.74 0)
+      (effects (font (size 1.27 1.27)) hide)
+    )
+    (property "Value" "+5V" (at 46.99 69.85 0)
+      (effects (font (size 1.27 1.27)))
+    )
+    (property "Footprint" "Diode_THT:D_P600_R-6_P20.00mm_Horizontal" (at 46.99 74.93 0)
+      (effects (font (size 1.27 1.27)) hide)
+    )
+    (property "Datasheet" "" (at 46.99 74.93 0)
+      (effects (font (size 1.27 1.27)) hide)
+    )
+    (pin "1")
+    (instances
+      (project "NMEA-2000-BUS-Voltage"
+        (path "/2ad9a196-bb2f-4407-b356-e110a1476183"
+          (reference "#PWR03") (unit 1)
+        )
+      )
+    )
+  )
   (sheet_instances
     (path "/" (page "1"))

Commit message: Added Potential Divider
Parts:
- added R1: 10k, symbol Device:R
- added R2: 1k5, symbol Device:R
- added R3: 1k, symbol Device:R
- added R4: 330R, symbol Device:R
Connections:
- net A0: now also R1.2, R2.1
- net GND: now also R4.2
- new net: R2.2, R3.1
- new net: R3.2, R4.1
- new net +12V: R1.1
Changed lines of the file:
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@@
 (kicad_sch (version 20230121) (generator eeschema)
   (paper "A4")
+  (junction (at 96.52 80.01) (diameter 0) (color 0 0 0 0)
+  )
   (no_connect (at 64.77 102.87))
   (no_connect (at 64.77 87.63))
@@
     (stroke (width 0) (type default))
   )
+  (wire (pts (xy 96.52 110.49) (xy 96.52 113.03))
+    (stroke (width 0) (type default))
+  )
   (wire (pts (xy 59.69 90.17) (xy 64.77 90.17))
     (stroke (width 0) (type default))
   )
+  (wire (pts (xy 91.44 80.01) (xy 96.52 80.01))
+    (stroke (width 0) (type default))
+  )
   (wire (pts (xy 64.77 105.41) (xy 59.69 105.41))
     (stroke (width 0) (type default))
   )
+  (wire (pts (xy 96.52 100.33) (xy 96.52 102.87))
+    (stroke (width 0) (type default))
+  )
   (wire (pts (xy 64.77 97.79) (xy 59.69 97.79))
     (stroke (width 0) (type default))
@@
     (stroke (width 0) (type default))
   )
+  (wire (pts (xy 96.52 90.17) (xy 96.52 92.71))
+    (stroke (width 0) (type default))
+  )
   (wire (pts (xy 64.77 100.33) (xy 59.69 100.33))
     (stroke (width 0) (type default))
@@
     (stroke (width 0) (type default))
   )
+  (wire (pts (xy 96.52 67.31) (xy 96.52 69.85))
+    (stroke (width 0) (type default))
+  )
+  (wire (pts (xy 96.52 77.47) (xy 96.52 80.01))
+    (stroke (width 0) (type default))
+  )
   (wire (pts (xy 59.69 85.09) (xy 64.77 85.09))
     (stroke (width 0) (type default))
   )
   (wire (pts (xy 64.77 102.87) (xy 59.69 102.87))
+    (stroke (width 0) (type default))
+  )
+  (wire (pts (xy 96.52 80.01) (xy 96.52 82.55))
     (stroke (width 0) (type default))
   )
@@
   (label "A0" (at 64.77 85.09 180) (fields_autoplaced)
     (effects (font (size 1.27 1.27)) (justify right bottom))
+  )
+  (label "A0" (at 91.44 80.01 0) (fields_autoplaced)
+    (effects (font (size 1.27 1.27)) (justify left bottom))
   )
   (label "FLS" (at 64.77 95.25 180) (fields_autoplaced)
@@
     )
   )
+  (symbol (lib_id "power:GND") (at 96.52 113.03 0) (unit 1)
+    (in_bom yes) (on_board yes) (dnp no) (fields_autoplaced)
+    (property "Reference" "#PWR05" (at 96.52 119.38 0)
+      (effects (font (size 1.27 1.27)) hide)
+    )
+    (property "Value" "GND" (at 96.52 118.11 0)
+      (effects (font (size 1.27 1.27)))
+    )
+    (property "Footprint" "" (at 96.52 113.03 0)
+      (effects (font (size 1.27 1.27)) hide)
+    )
+    (property "Datasheet" "" (at 96.52 113.03 0)
+      (effects (font (size 1.27 1.27)) hide)
+    )
+    (pin "1")
+    (instances
+      (project "NMEA-2000-BUS-Voltage"
+        (path "/2ad9a196-bb2f-4407-b356-e110a1476183"
+          (reference "#PWR05") (unit 1)
+        )
+      )
+    )
+  )
   (symbol (lib_id "power:+3V3") (at 52.07 74.93 0) (unit 1)
     (in_bom yes) (on_board yes) (dnp no) (fields_autoplaced)
@@
     )
   )
+  (symbol (lib_id "Device:R") (at 96.52 96.52 0) (unit 1)
+    (in_bom yes) (on_board yes) (dnp no) (fields_autoplaced)
+    (property "Reference" "R3" (at 99.06 95.25 0)
+      (effects (font (size 1.27 1.27)) (justify left))
+    )
+    (property "Value" "1k" (at 99.06 97.79 0)
+      (effects (font (size 1.27 1.27)) (justify left))
+    )
+    (property "Footprint" "" (at 94.742 96.52 90)
+      (effects (font (size 1.27 1.27)) hide)
+    )
+    (property "Datasheet" "~" (at 96.52 96.52 0)
+      (effects (font (size 1.27 1.27)) hide)
+    )
+    (pin "1")
+    (pin "2")
+    (instances
+      (project "NMEA-2000-BUS-Voltage"
+        (path "/2ad9a196-bb2f-4407-b356-e110a1476183"
+          (reference "R3") (unit 1)
+        )
+      )
+    )
+  )
   (symbol (lib_id "power:+5V") (at 46.99 74.93 0) (unit 1)
     (in_bom yes) (on_board yes) (dnp no) (fields_autoplaced)
@@
         )
       )
+    )
+  )
+  (symbol (lib_id "Device:R") (at 96.52 73.66 0) (unit 1)
+    (in_bom yes) (on_board yes) (dnp no) (fields_autoplaced)
+    (property "Reference" "R1" (at 99.06 72.39 0)
+      (effects (font (size 1.27 1.27)) (justify left))
+    )
+    (property "Value" "10k" (at 99.06 74.93 0)
+      (effects (font (size 1.27 1.27)) (justify left))
+    )
+    (property "Footprint" "" (at 94.742 73.66 90)
+      (effects (font (size 1.27 1.27)) hide)
+    )
+    (property "Datasheet" "~" (at 96.52 73.66 0)
+      (effects (font (size 1.27 1.27)) hide)
+    )
+    (pin "1")
+    (pin "2")
+    (instances
+      (project "NMEA-2000-BUS-Voltage"
+        (path "/2ad9a196-bb2f-4407-b356-e110a1476183"
+          (reference "R1") (unit 1)
+        )
+      )
+    )
+  )
+  (symbol (lib_id "power:+12V") (at 96.52 67.31 0) (unit 1)
+    (in_bom yes) (on_board yes) (dnp no) (fields_autoplaced)
+    (property "Reference" "#PWR04" (at 96.52 71.12 0)
+      (effects (font (size 1.27 1.27)) hide)
+    )
+    (property "Value" "+12V" (at 96.52 62.23 0)
+      (effects (font (size 1.27 1.27)))
+    )
+    (property "Footprint" "" (at 96.52 67.31 0)
+      (effects (font (size 1.27 1.27)) hide)
+    )
+    (property "Datasheet" "" (at 96.52 67.31 0)
+      (effects (font (size 1.27 1.27)) hide)
+    )
+    (pin "1")
+    (instances
+      (project "NMEA-2000-BUS-Voltage"
+        (path "/2ad9a196-bb2f-4407-b356-e110a1476183"
+          (reference "#PWR04") (unit 1)
+        )
+      )
+    )
+  )
+  (symbol (lib_id "Device:R") (at 96.52 106.68 0) (unit 1)
+    (in_bom yes) (on_board yes) (dnp no) (fields_autoplaced)
+    (property "Reference" "R4" (at 99.06 105.41 0)
+      (effects (font (size 1.27 1.27)) (justify left))
+    )
+    (property "Value" "330R" (at 99.06 107.95 0)
+      (effects (font (size 1.27 1.27)) (justify left))
+    )
+    (property "Footprint" "" (at 94.742 106.68 90)
+      (effects (font (size 1.27 1.27)) hide)
+    )
+    (property "Datasheet" "~" (at 96.52 106.68 0)
+      (effects (font (size 1.27 1.27)) hide)
+    )
+    (pin "1")
+    (pin "2")
+    (instances
+      (project "NMEA-2000-BUS-Voltage"
+        (path "/2ad9a196-bb2f-4407-b356-e110a1476183"
+          (reference "R4") (unit 1)
+        )
+      )
+    )
+  )
+  (symbol (lib_id "Device:R") (at 96.52 86.36 0) (unit 1)
+    (in_bom yes) (on_board yes) (dnp no) (fields_autoplaced)
+    (property "Reference" "R2" (at 99.06 85.09 0)
+      (effects (font (size 1.27 1.27)) (justify left))
+    )
+    (property "Value" "1k5" (at 99.06 87.63 0)
+      (effects (font (size 1.27 1.27)) (justify left))
+    )
+    (property "Footprint" "" (at 94.742 86.36 90)
+      (effects (font (size 1.27 1.27)) hide)
+    )
+    (property "Datasheet" "~" (at 96.52 86.36 0)
+      (effects (font (size 1.27 1.27)) hide)
+    )
+    (pin "1")
+    (pin "2")
+    (instances
+      (project "NMEA-2000-BUS-Voltage"
+        (path "/2ad9a196-bb2f-4407-b356-e110a1476183"
+          (reference "R2") (unit 1)
+        )
+      )

Commit message: Added Flash Button
Parts:
- added SW1: SW_Push, symbol Switch:SW_Push
Connections:
- net FLS: now also SW1.1
- net GND: now also SW1.2
Changed lines of the file:
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@@
+    (stroke (width 0) (type default))
+  )
+  (wire (pts (xy 124.46 64.77) (xy 124.46 59.69))
     (stroke (width 0) (type default))
   )
@@
   )
   (wire (pts (xy 64.77 107.95) (xy 59.69 107.95))
+    (stroke (width 0) (type default))
+  )
+  (wire (pts (xy 124.46 74.93) (xy 124.46 77.47))
     (stroke (width 0) (type default))
   )
@@
   (label "RX" (at 34.29 95.25 0) (fields_autoplaced)
     (effects (font (size 1.27 1.27)) (justify left bottom))
+  )
+  (label "FLS" (at 124.46 59.69 270) (fields_autoplaced)
+    (effects (font (size 1.27 1.27)) (justify right bottom))
   )
   (label "D1" (at 64.77 90.17 180) (fields_autoplaced)
@@
     )
   )
+  (symbol (lib_id "power:GND") (at 124.46 77.47 0) (unit 1)
+    (in_bom yes) (on_board yes) (dnp no) (fields_autoplaced)
+    (property "Reference" "#PWR06" (at 124.46 83.82 0)
+      (effects (font (size 1.27 1.27)) hide)
+    )
+    (property "Value" "GND" (at 124.46 82.55 0)
+      (effects (font (size 1.27 1.27)))
+    )
+    (property "Footprint" "" (at 124.46 77.47 0)
+      (effects (font (size 1.27 1.27)) hide)
+    )
+    (property "Datasheet" "" (at 124.46 77.47 0)
+      (effects (font (size 1.27 1.27)) hide)
+    )
+    (pin "1")
+    (instances
+      (project "NMEA-2000-BUS-Voltage"
+        (path "/2ad9a196-bb2f-4407-b356-e110a1476183"
+          (reference "#PWR06") (unit 1)
+        )
+      )
+    )
+  )
   (symbol (lib_id "Device:R") (at 96.52 96.52 0) (unit 1)
     (in_bom yes) (on_board yes) (dnp no) (fields_autoplaced)
@@
         )
       )
+    )
+  )
+  (symbol (lib_id "Switch:SW_Push") (at 124.46 69.85 270) (unit 1)
+    (in_bom yes) (on_board yes) (dnp no) (fields_autoplaced)
+    (property "Reference" "SW1" (at 128.27 68.58 90)
+      (effects (font (size 1.27 1.27)) (justify left))
+    )
+    (property "Value" "SW_Push" (at 128.27 71.12 90)
+      (effects (font (size 1.27 1.27)) (justify left))
+    )
+    (property "Footprint" "" (at 129.54 69.85 0)
+      (effects (font (size 1.27 1.27)) hide)
+    )
+    (property "Datasheet" "~" (at 129.54 69.85 0)
+      (effects (font (size 1.27 1.27)) hide)
+    )
+    (pin "1")
+    (pin "2")
+    (instances
+      (project "NMEA-2000-BUS-Voltage"
+        (path "/2ad9a196-bb2f-4407-b356-e110a1476183"
+          (reference "SW1") (unit 1)
+        )
+      )
