File: Electrical/NMEA-2000-Bus-Voltage-sensor.kicad_sch (KiCad schematic)
At the start: 51 parts, among them IC1 ADS131M08, J10 Conn_01x02, J11 Conn_01x05, J12 Conn_01x02, J13 Conn_01x02, J5 Conn_01x05, J6 Conn_01x05, J7 Conn_01x02, J8 Conn_01x02, J9 Conn_01x02, K1 Relay_SPDT, K2 Relay_SPDT, Q1 IRFZ44N, Q2 IRFZ44N, U6 ADR4533, Y3 20kHz Crystal

Commit message: Cleaned Up Project Updated BOM Updated Naming
Other:
- company: (none) -> Johannes Höllwerth
- title: Bus Power -> N2k Bus Power
Changed lines of the file:
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@@
 	(paper "A4")
 	(title_block
-		(title "Bus Power")
-		(date "2024-06-12")
-		(rev "2")
+		(title "N2k Bus Power")
+		(date "2024-07-06")
+		(rev "3")
+		(company "Johannes Höllwerth")
+		(comment 2 "Sensors and Relays")
 	)
 	(junction
@@
 		)
 		(instances
-			(project ""
+			(project "NMEA-2000-BUS-Voltage"
 				(path "/2ad9a196-bb2f-4407-b356-e110a1476183/f2085319-9271-4df7-bfa7-865ab61d6adc"
 					(reference "J11")
@@
 		)
 		(instances
-			(project ""
+			(project "NMEA-2000-BUS-Voltage"
 				(path "/2ad9a196-bb2f-4407-b356-e110a1476183/f2085319-9271-4df7-bfa7-865ab61d6adc"
 					(reference "J10")
@@
 		)
 		(instances
-			(project ""
+			(project "NMEA-2000-BUS-Voltage"
 				(path "/2ad9a196-bb2f-4407-b356-e110a1476183/f2085319-9271-4df7-bfa7-865ab61d6adc"
 					(reference "JP7")
